File: pcb/naicha68.kicad_pcb (KiCad board)
At the start: 2 copper layers, 342.9 x 96.7 mm, 147 parts, among them J1 Conn_01x05_Socket, J2 Conn_01x02_Pin, SW1 SW_Push, SW10 SW_Push, SW11 SW_Push, SW12 SW_Push, SW13 SW_Push, SW14 SW_Push, SW15 SW_Push, SW16 SW_Push, SW17 SW_Push, SW18 SW_Push, SW19 SW_Push, SW2 SW_Push, SW20 SW_Push, SW21 SW_Push, SW22 SW_Push, SW23 SW_Push, SW24 SW_Push, SW25 SW_Push, SW26 SW_Push, SW27 SW_Push, SW28 SW_Push, SW29 SW_Push, SW3 SW_Push, SW30 SW_Push, SW31 SW_Push, SW32 SW_Push, SW33 SW_Push, SW34 SW_Push, SW35 SW_Push, SW36 SW_Push, SW37 SW_Push, SW38 SW_Push, SW39 SW_Push, SW4 SW_Push, SW40 SW_Push, SW41 SW_Push, SW42 SW_Push, SW43 SW_Push, SW44 SW_Push, SW45 SW_Push, SW46 SW_Push, SW47 SW_Push, SW48 SW_Push, SW49 SW_Push, SW5 SW_Push, SW50 SW_Push, SW51 SW_Push, SW52 SW_Push, SW53 SW_Push, SW54 SW_Push, SW55 SW_Push, SW56 SW_Push, SW57 SW_Push, SW58 SW_Push, SW59 SW_Push, SW6 SW_Push, SW60 SW_Push, SW61 SW_Push, SW62 SW_Push, SW63 SW_Push, SW64 SW_Push, SW65 SW_Push, SW66 SW_Push, SW67 SW_Push, SW68 SW_Push, SW7 SW_Push, SW8 SW_Push, SW9 SW_Push, U2 PCA9555D, U3 PCA9555D, U4 XIAO-nRF52840-SMD

Commit message: new pcb udpates
Parts:
- J1: value Conn_01x05_Socket -> Conn_01x04_Socket; footprint Connector_PinHeader_2.54mm:PinHeader_1x05_P2.54mm_Vertical -> Connector_PinHeader_2.54mm:PinHeader_1x04_P2.54mm_Vertical
- moved J2 2.00 mm to (330.5, 151.0)
- moved J1 1.73 mm to (349.5, 163.8)
- moved R1 1.50 mm to (342.4, 145.0)
- moved R2 1.50 mm to (338.6, 145.0)
- moved U4 1.49 mm to (335.5, 131.0)
Connections:
- J1 pad 1: MISO -> SDA
- J1 pad 2: SCK -> VCC
- J1 pad 3: VCC -> GND
- J1 pad 4: GND -> SCL
Routing:
- net MISO: track 52.8 -> 0.00 mm, vias 1 -> 0
- net SCK: track 51.1 -> 0.00 mm, vias 1 -> 0
- net CS: track 50.5 -> 0.00 mm
- net COL13: track 382.6 -> 362.5 mm
- net COL11: track 282.7 -> 299.7 mm
- net COL9: track 329.7 -> 345.7 mm, vias 4 -> 3
- net ROW1: track 464.5 -> 476.8 mm, vias 13 -> 14
- net ROW3: track 352.6 -> 364.3 mm
- net COL7: track 207.7 -> 217.9 mm
- net SDA: track 91.1 -> 101.0 mm
- net SCL: track 90.6 -> 98.3 mm
- net COL1: track 148.6 -> 141.0 mm
- net COL10: track 267.8 -> 260.3 mm
- net COL3: track 131.5 -> 138.8 mm, vias 1 -> 2
- net VCC: track 119.2 -> 112.2 mm, vias 2 -> 1
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Other:
- board size 342.9 x 96.7 mm -> 342.9 x 95.2 mm
